File: hardware/kicad/misrc.kicad_sch (KiCad schematic)
At the start: 24 parts, among them J1 Conn_01x01_Shielded, J2 Conn_01x08_Socket, J3 GPIFII_J6, J4 GPIFII_J7, SW1 SW_Push, U1 4043, U2 74VHC541, U3 74VHC541, U4 74VHC541, U5 74VHC541

Commit message: new hardware revision
Parts:
- added C31: 1µ, Capacitor_SMD:C_0805_2012Metric, symbol Device:C
- added SW2: SW_DIP_x01, Button_Switch_SMD:SW_DIP_SPSTx01_Slide_6.7x4.1mm_W8.61mm_P2.54mm_LowProfile, symbol Switch:SW_DIP_x01
- added X1: 40M, Oscillator:Oscillator_SMD_EuroQuartz_XO53-4Pin_5.0x3.2mm, symbol Oscillator:XO53
Connections:
- net GND: now also J3.33 (GND), C31.2, SW2.1, X1.2 (GND)
- net Input_ADC_CH1/CLK: now also X1.3 (OUT)
- net VDD: now also C31.1, X1.4 (V+)
- new net: SW2.2, X1.1 (EN)
Other:
- moved on the sheet: J1
