File: hardware/kicad/power_supply.kicad_sch (KiCad schematic)
At the start: 29 parts, among them Q1 FZT690B, Q2 FZT790A, U6 TPS60401, U7 ADP7156ARDZ

Commit message: new hardware revision
Parts:
- added C27: 1n, Capacitor_SMD:C_0805_2012Metric, symbol Device:C
- added C28: 10µ, Capacitor_SMD:C_0805_2012Metric, symbol Device:C
- added C29, C30: 1µ, Capacitor_SMD:C_0805_2012Metric, symbol Device:C
Connections:
- net +5VA: now also C30.1
- net -5VA: now also C29.1
- net GND: now also C27.1, C28.1, C29.2, C30.2
- net at L2.1, U6.1 (VOUT): now also C27.2, C28.2
Other:
- title: FX3 USB3 ADC -> MISRC
- moved on the sheet: C10, C11, C12, C13, C14, C15, C16, C17, C18, C19, C20, C21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

Commit message: Updated annonation on the PCB, added gerbers, PDFs and BOM
Parts:
- C27: value 1n -> 1n/1
Other:
- note added: "Capacitor values with "/1" suffix indicate parts that are required to be class 1 ceramic material"
Changed lines of the file:
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@@
     (stroke (width 0) (type default))
+  )
+  (text "Capacitor values with \"/1\" suffix indicate parts that are required to be class 1 ceramic material"
+    (at 20.32 24.13 0)
+    (effects (font (size 1.27 1.27)) (justify left bottom))
   )
   (symbol (lib_id "power:GND") (at 67.31 52.07 0) (unit 1)
@@
       (effects (font (size 1.27 1.27)) (justify left))
     )
-    (property "Value" "1n" (at 59.69 73.66 0)
-      (effects (font (size 1.27 1.27)) (justify left))
-    )
+    (property "Value" "1n/1" (at 59.69 73.66 0)
+      (effects (font (size 1.27 1.27)) (justify left))
+    )
