File: hardware/kicad/v1.5/misrc_v1.5.kicad_pcb (KiCad board)
At the start: 2 copper layers, 146.2 x 72.6 mm, 194 parts, among them J1 Conn_01x01_Shielded, J2 Conn_01x08_Socket, J201 DOSIN-801-0050, J3 GPIFII_J6, J4 GPIFII_J7, Q1 FZT690B, Q101 CMPT5179, Q102 CMPT5179, Q2 FZT790A, Q201 CMPT5179, Q202 CMPT5179, SW1 SW_Push, SW101 SW_DIP_x04, SW102 SW_DIP_x03, SW103 SW_DIP_x03, SW104 SW_DIP_x03, SW105 SW_DIP_x02, SW2 SW_DIP_x01, SW201 SW_DIP_x04, SW202 SW_DIP_x03, SW203 SW_DIP_x03, SW204 SW_DIP_x03, SW205 SW_DIP_x02, U1 4043, U101 AD8138ARZ, U102 AD9235, U2 74VHC541, U201 AD8138ARZ, U202 AD9235, U3 74VHC541, U4 74VHC541, U5 74VHC541, U6 TPS60401, U7 ADP7156ARDZ, X1 40M

Commit message: Fix J201 pad path, causing production issues with fabs
Connections:
- J201 pad 1: Net-(J101-Signal) -> Net-(J201-Signal)
Changed lines of the file:
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@@
 			(layers "*.Cu" "*.Mask")
 			(remove_unused_layers no)
-			(net 50 "Net-(J101-Signal)")
+			(net 66 "Net-(J201-Signal)")
 		)
 		(pad "2" thru_hole circle
