File: hardware/kicad/dev/audio_adc.kicad_sch (KiCad schematic)
At the start: 37 parts, among them J301 KLP42X-61-WW_RR, U301 PCM1802DBR, U401 PCM1802DBR

Commit message: repositioning of parts for more case options
Connections:
- net IN1_L: now also R402.1; no longer R301.1
- net IN1_R: now also R401.1; no longer R302.1
- net IN2_L: now also R302.1; no longer R401.1
- net IN2_R: now also R301.1; no longer R402.1
- net at C304.2, C305.2: now also U301.1 (VINL); no longer U301.2 (VINR)
- net at C302.2, C303.2: now also U301.2 (VINR); no longer U301.1 (VINL)
- net at C404.2, C405.2: now also U401.1 (VINL); no longer U401.2 (VINR)
- net at C402.2, C403.2: now also U401.2 (VINR); no longer U401.1 (VINL)
Other:
- moved on the sheet: C302, C303, C304, C305, C402, C403, C404, C405, R301, R302, R303, R304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
