File: hardware/kicad/dev/input_adc_CH2.kicad_sch (KiCad schematic)
At the start: 91 parts, among them J201 BNC_Rosenberger, J201/2 Conn_01x01_Shielded, J201/3 Conn_Coaxial, SW201 SW_DIP_x04, SW202 SW_DIP_x03, SW203 SW_DIP_x04, SW204 SW_DIP_x03, U201 AD8138ARZ, U202 AD9235

Commit message: Silkscreen updates
Parts:
- R202: value 300B -> 100B; LCSC Part # C705763 -> C122970; Manufacturer_Part_Number RT0603BRD07300RL -> RT0603BRD07100RL
- R203: value 100B -> 300B; LCSC Part # C122970 -> C705763; Manufacturer_Part_Number RT0603BRD07100RL -> RT0603BRD07300RL
- R206: value 150B -> 49R9B; LCSC Part # C705726 -> C861434; Manufacturer_Part_Number RT0603BRD07150RL -> RT0603BRD0749R9L
- R207: value 49R9B -> 150B; LCSC Part # C861434 -> C705726; Manufacturer_Part_Number RT0603BRD0749R9L -> RT0603BRD07150RL
Changed lines of the file:
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@@
 	(title_block
 		(title "MISRC")
-		(date "2025-08-10")
+		(date "2025-10-10")
 		(rev "2.5")
 		(comment 1 "Analog input + ADC")
@@
 			)
 		)
-		(property "Value" "49R9B"
+		(property "Value" "150B"
 			(at 83.312 71.882 90)
 			(effects
@@
 			)
 		)
-		(property "Manufacturer_Part_Number" "RT0603BRD0749R9L"
+		(property "Manufacturer_Part_Number" "RT0603BRD07150RL"
 			(at 85.09 78.74 0)
 			(effects
@@
 			)
 		)
-		(property "LCSC Part #" "C861434"
+		(property "LCSC Part #" "C705726"
 			(at 85.09 78.74 90)
 			(effects
@@
 			)
 		)
-		(property "Value" "300B"
+		(property "Value" "100B"
 			(at 52.07 64.77 90)
 			(effects
@@
 			)
 		)
-		(property "Manufacturer_Part_Number" "RT0603BRD07300RL"
+		(property "Manufacturer_Part_Number" "RT0603BRD07100RL"
 			(at 52.07 59.69 0)
 			(effects
@@
 			)
 		)
-		(property "LCSC Part #" "C705763"
+		(property "LCSC Part #" "C122970"
 			(at 52.07 59.69 90)
 			(effects
@@
 			)
 		)
-		(property "Value" "100B"
+		(property "Value" "300B"
 			(at 55.88 64.77 90)
 			(effects
@@
 			)
 		)
-		(property "Manufacturer_Part_Number" "RT0603BRD07100RL"
+		(property "Manufacturer_Part_Number" "RT0603BRD07300RL"
 			(at 55.88 59.69 0)
 			(effects
@@
 			)
 		)
-		(property "LCSC Part #" "C122970"
+		(property "LCSC Part #" "C705763"
 			(at 55.88 59.69 90)
 			(effects
@@
 			)
 		)
-		(property "Value" "150B"
+		(property "Value" "49R9B"
 			(at 79.248 72.39 90)
 			(effects
@@
 			)
 		)
-		(property "Manufacturer_Part_Number" "RT0603BRD07150RL"
+		(property "Manufacturer_Part_Number" "RT0603BRD0749R9L"
 			(at 81.28 78.74 0)
 			(effects
@@
 			)
 		)
-		(property "LCSC Part #" "C705726"
+		(property "LCSC Part #" "C861434"
 			(at 81.28 78.74 90)
 			(effects
