File: hardware/kicad/dev/input_adc.kicad_sch (KiCad schematic)
At the start: 91 parts, among them J101 BNC_Rosenberger, J101/2 Conn_01x01_Shielded, J101/3 Conn_Coaxial, SW101 SW_DIP_x04, SW102 SW_DIP_x03, SW103 SW_DIP_x04, SW104 SW_DIP_x03, U101 AD8138ARZ, U102 AD9235

Commit message: Silkscreen updates
Parts:
- R102: value 300B -> 100B; LCSC Part # C705763 -> C122970; Manufacturer_Part_Number RT0603BRD07300RL -> RT0603BRD07100RL
- R103: value 100B -> 300B; LCSC Part # C122970 -> C705763; Manufacturer_Part_Number RT0603BRD07100RL -> RT0603BRD07300RL
- R106: value 150B -> 49R9B; LCSC Part # C705726 -> C861434; Manufacturer_Part_Number RT0603BRD07150RL -> RT0603BRD0749R9L
- R107: value 49R9B -> 150B; LCSC Part # C861434 -> C705726; Manufacturer_Part_Number RT0603BRD0749R9L -> RT0603BRD07150RL
Changed lines of the file:
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@@
 	(title_block
 		(title "MISRC")
-		(date "2025-08-10")
+		(date "2025-10-10")
 		(rev "2.5")
 		(comment 1 "Analog input + ADC")
@@
 			)
 		)
-		(property "Value" "150B"
+		(property "Value" "49R9B"
 			(at 80.01 72.39 90)
 			(effects
@@
 			)
 		)
-		(property "Manufacturer_Part_Number" "RT0603BRD07150RL"
+		(property "Manufacturer_Part_Number" "RT0603BRD0749R9L"
 			(at 81.28 78.74 0)
 			(effects
@@
 			)
 		)
-		(property "LCSC Part #" "C705726"
+		(property "LCSC Part #" "C861434"
 			(at 81.28 78.74 90)
 			(effects
@@
 			)
 		)
-		(property "Value" "300B"
+		(property "Value" "100B"
 			(at 52.07 64.77 90)
 			(effects
@@
 			)
 		)
-		(property "Manufacturer_Part_Number" "RT0603BRD07300RL"
+		(property "Manufacturer_Part_Number" "RT0603BRD07100RL"
 			(at 52.07 59.69 0)
 			(effects
@@
 			)
 		)
-		(property "LCSC Part #" "C705763"
+		(property "LCSC Part #" "C122970"
 			(at 52.07 59.69 90)
 			(effects
@@
 			)
 		)
-		(property "Value" "49R9B"
+		(property "Value" "150B"
 			(at 83.82 72.39 90)
 			(effects
@@
 			)
 		)
-		(property "Manufacturer_Part_Number" "RT0603BRD0749R9L"
+		(property "Manufacturer_Part_Number" "RT0603BRD07150RL"
 			(at 85.09 78.74 0)
 			(effects
@@
 			)
 		)
-		(property "LCSC Part #" "C861434"
+		(property "LCSC Part #" "C705726"
 			(at 85.09 78.74 90)
 			(effects
@@
 			)
 		)
-		(property "Value" "100B"
+		(property "Value" "300B"
 			(at 55.88 64.77 90)
 			(effects
@@
 			)
 		)
-		(property "Manufacturer_Part_Number" "RT0603BRD07100RL"
+		(property "Manufacturer_Part_Number" "RT0603BRD07300RL"
 			(at 55.88 59.69 0)
 			(effects
@@
 			)
 		)
-		(property "LCSC Part #" "C122970"
+		(property "LCSC Part #" "C705763"
 			(at 55.88 59.69 90)
 			(effects

Commit message: changed pot direction
Connections:
- net +5VA: now also RV101.3; no longer RV101.1
- net -5VA: now also RV101.1; no longer RV101.3
Changed lines of the file:
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@@
 	(title_block
 		(title "MISRC")
-		(date "2025-10-10")
+		(date "2025-10-12")
 		(rev "2.5")
 		(comment 1 "Analog input + ADC")
@@
 		(lib_id "Device:R_Potentiometer")
 		(at 48.26 105.41 0)
-		(mirror x)
 		(unit 1)
 		(exclude_from_sim no)
@@
 		)
 		(property "Value" "10k"
-			(at 50.8 107.95 90)
+			(at 50.546 107.95 90)
 			(effects
 				(font
@@
 		)
 		(instances
-			(project "MISRC_v3.0"
+			(project "misrc_v2.5"
 				(path "/bc796fa4-76ff-4554-a44c-2597c6c5788e/f3827713-3b6b-4193-bf1c-3910c26c6fe9"
 					(reference "RV101")

Commit message: updated bom
Parts:
- C101: Manufacturer_Part_Number EMK325ABJ107MM-P -> EMK325ABJ107MM-P
- C118, C119: LCSC Part # C519563 -> C1864402; Manufacturer_Part_Number CC0603FRNPO9BN391 -> GCM1885C2A391FA16D
- C132, C133: LCSC Part # C3895655 -> C3859396; Manufacturer_Name (none) -> Murata; Manufacturer_Part_Number 0603N361F500CT -> GCM1885C2A361FA16D; Mouser Part Number (none) -> 81-GCM1885C2A361FA6D
- C141: Mouser Part Number (none) -> 80-C1812C944J5JLCLTU
- L101, L102: LCSC Part # C346452 -> C2042960; Manufacturer_Part_Number FEC1008CP-R62G-LRH -> LQW2UASR62F00L; Max Tolerance 2% -> 1%
- L103, L104, L105, L106: LCSC Part # C346451 -> C907989; Manufacturer_Part_Number FEC1008CP-R56G-LRH -> LQW2UASR56F00L; Max Tolerance 2% -> 1%
- R107: LCSC Part # C705726 -> C425408; Manufacturer_Part_Number RT0603BRD07150RL -> TC0325B1500T5F
- R119, R120, R121, R122: LCSC Part # C326724 -> C2989449; Manufacturer_Part_Number RT0603BRD0747RL -> TC0325B470JT5F
- SW101, SW103: Mouser Part Number (none) -> 611-SDA04H1SBDR
Changed lines of the file:
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@@
 			)
 		)
-		(property "Manufacturer_Part_Number" "RT0603BRD0747RL"
+		(property "Manufacturer_Part_Number" "TC0325B470JT5F"
 			(at 191.77 69.85 0)
 			(effects
@@
 			)
 		)
-		(property "LCSC Part #" "C326724"
+		(property "LCSC Part #" "C2989449"
 			(at 191.77 69.85 90)
 			(effects
@@
 			)
 		)
-		(property "Manufacturer_Part_Number" "FEC1008CP-R62G-LRH"
+		(property "Manufacturer_Part_Number" "LQW2UASR62F00L"
 			(at 142.24 69.85 90)
 			(effects
@@
 			)
 		)
-		(property "LCSC Part #" "C346452"
+		(property "LCSC Part #" "C2042960"
 			(at 142.24 69.85 90)
 			(effects
@@
 			)
 		)
-		(property "Max Tolerance" "2%"
+		(property "Max Tolerance" "1%"
 			(at 142.24 69.85 90)
 			(effects
@@
 			)
 		)
-		(property "Manufacturer_Part_Number" "RT0603BRD0747RL"
+		(property "Manufacturer_Part_Number" "TC0325B470JT5F"
 			(at 130.81 69.85 0)
 			(effects
@@
 			)
 		)
-		(property "LCSC Part #" "C326724"
+		(property "LCSC Part #" "C2989449"
 			(at 130.81 69.85 90)
 			(effects
@@
 			)
 		)
-		(property "Manufacturer_Part_Number" "FEC1008CP-R62G-LRH"
+		(property "Manufacturer_Part_Number" "LQW2UASR62F00L"
 			(at 142.24 64.77 90)
 			(effects
@@
 			)
 		)
-		(property "LCSC Part #" "C346452"
+		(property "LCSC Part #" "C2042960"
 			(at 142.24 64.77 90)
 			(effects
@@
 			)
 		)
-		(property "Max Tolerance" "2%"
+		(property "Max Tolerance" "1%"
 			(at 142.24 64.77 90)
 			(effects
@@
 			)
 		)
-		(property "Manufacturer_Part_Number" "CC0603FRNPO9BN391"
+		(property "Manufacturer_Part_Number" "GCM1885C2A391FA16D"
 			(at 153.67 55.88 0)
 			(effects
@@
 			)
 		)
-		(property "LCSC Part #" "C519563"
+		(property "LCSC Part #" "C1864402"
 			(at 153.67 55.88 0)
 			(effects
@@
 			)
 		)
-		(property "Manufacturer_Part_Number" "0603N361F500CT"
+		(property "Manufacturer_Part_Number" "GCM1885C2A361FA16D"
 			(at 172.72 78.74 0)
 			(effects
@@
 			)
 		)
-		(property "LCSC Part #" "C3895655"
+		(property "LCSC Part #" "C3859396"
 			(at 172.72 78.74 0)
 			(effects
@@
 			)
 		)
+		(property "Manufacturer_Name" "Murata"
+			(at 172.72 78.74 0)
+			(effects
+				(font
+					(size 1.27 1.27)
+				)
+				(hide yes)
+			)
+		)
+		(property "Mouser Part Number" "81-GCM1885C2A361FA6D"
+			(at 172.72 78.74 0)
+			(effects
+				(font
+					(size 1.27 1.27)
+				)
+				(hide yes)
+			)
+		)
 		(pin "1"
 		)
@@
 			)
 		)
-		(property "Manufacturer_Part_Number" "FEC1008CP-R56G-LRH"
+		(property "Manufacturer_Part_Number" "LQW2UASR56F00L"
 			(at 179.07 64.77 90)
 			(effects
@@
 			)
 		)
-		(property "LCSC Part #" "C346451"
+		(property "LCSC Part #" "C907989"
 			(at 179.07 64.77 90)
 			(effects
@@
 			)
 		)
-		(property "Max Tolerance" "2%"
+		(property "Max Tolerance" "1%"
 			(at 179.07 64.77 90)
 			(effects
@@
 			)
 		)
-		(property "Manufacturer_Part_Number" "FEC1008CP-R56G-LRH"
+		(property "Manufacturer_Part_Number" "LQW2UASR56F00L"
 			(at 166.37 64.77 90)
 			(effects
@@
 			)
 		)
-		(property "LCSC Part #" "C346451"
+		(property "LCSC Part #" "C907989"
 			(at 166.37 64.77 90)
 			(effects
@@
 			)
 		)
-		(property "Max Tolerance" "2%"
+		(property "Max Tolerance" "1%"
 			(at 166.37 64.77 90)
 			(effects
@@
 			)
 		)
-		(property "Manufacturer_Part_Number" "0603N361F500CT"
+		(property "Manufacturer_Part_Number" "GCM1885C2A361FA16D"
 			(at 172.72 55.88 0)
 			(effects
@@
 			)
 		)
-		(property "LCSC Part #" "C3895655"
+		(property "LCSC Part #" "C3859396"
 			(at 172.72 55.88 0)
 			(effects
@@
 			)
 		)
+		(property "Manufacturer_Name" "Murata"
+			(at 172.72 55.88 0)
+			(effects
+				(font
+					(size 1.27 1.27)
+				)
+				(hide yes)
+			)
+		)
+		(property "Mouser Part Number" "81-GCM1885C2A361FA6D"
+			(at 172.72 55.88 0)
+			(effects
+				(font
+					(size 1.27 1.27)
+				)
+				(hide yes)
+			)
+		)
 		(pin "1"
 		)
@@
 			)
 		)
+		(property "Mouser Part Number" "80-C1812C944J5JLCLTU"
+			(at 63.5 73.66 90)
+			(effects
+				(font
+					(size 1.27 1.27)
+				)
+				(hide yes)
+			)
+		)
 		(pin "1"
 		)
@@
 			)
 		)
-		(property "Manufacturer_Part_Number" "RT0603BRD07150RL"
+		(property "Manufacturer_Part_Number" "TC0325B1500T5F"
 			(at 85.09 78.74 0)
 			(effects
@@
 			)
 		)
-		(property "LCSC Part #" "C705726"
+		(property "LCSC Part #" "C425408"
 			(at 85.09 78.74 90)
 			(effects
@@
 			)
 		)
-		(property "Manufacturer_Part_Number" "RT0603BRD0747RL"
+		(property "Manufacturer_Part_Number" "TC0325B470JT5F"
 			(at 130.81 64.77 0)
 			(effects
@@
 			)
 		)
-		(property "LCSC Part #" "C326724"
+		(property "LCSC Part #" "C2989449"
 			(at 130.81 64.77 90)
 			(effects
@@
 			)
 		)
-		(property "Manufacturer_Part_Number" "CC0603FRNPO9BN391"
+		(property "Manufacturer_Part_Number" "GCM1885C2A391FA16D"
 			(at 153.67 78.74 0)
 			(effects
@@
 			)
 		)
-		(property "LCSC Part #" "C519563"
+		(property "LCSC Part #" "C1864402"
 			(at 153.67 78.74 0)
 			(effects
@@
 			)
 		)
-		(property "Manufacturer_Part_Number" "FEC1008CP-R56G-LRH"
+		(property "Manufacturer_Part_Number" "LQW2UASR56F00L"
 			(at 166.37 69.85 90)
 			(effects
@@
 			)
 		)
-		(property "LCSC Part #" "C346451"
+		(property "LCSC Part #" "C907989"
 			(at 166.37 69.85 90)
 			(effects
@@
 			)
 		)
-		(property "Max Tolerance" "2%"
+		(property "Max Tolerance" "1%"
 			(at 166.37 69.85 90)
 			(effects
@@
 			)
 		)
+		(property "Mouser Part Number" "611-SDA04H1SBDR"
+			(at 119.38 45.72 90)
+			(effects
+				(font
+					(size 1.27 1.27)
+				)
+				(hide yes)
+			)
+		)
 		(pin "1"
 		)
@@
 			)
 		)
-		(property "Manufacturer_Part_Number" "RT0603BRD0747RL"
+		(property "Manufacturer_Part_Number" "TC0325B470JT5F"
 			(at 191.77 64.77 0)
 			(effects
@@
 			)
 		)
-		(property "LCSC Part #" "C326724"
+		(property "LCSC Part #" "C2989449"
 			(at 191.77 64.77 90)
 			(effects
@@
 			)
 		)
+		(property "Mouser Part Number" "611-SDA04H1SBDR"
+			(at 55.88 44.45 90)
+			(effects
+				(font
+					(size 1.27 1.27)
+				)
+				(hide yes)
+			)
+		)
 		(pin "1"
 		)
@@
 			)
 		)
-		(property "Manufacturer_Part_Number" " EMK325ABJ107MM-P"
+		(property "Manufacturer_Part_Number" "EMK325ABJ107MM-P"
 			(at 41.91 63.5 0)
 			(effects
@@
 			)
 		)
-		(property "Manufacturer_Part_Number" "FEC1008CP-R56G-LRH"
+		(property "Manufacturer_Part_Number" "LQW2UASR56F00L"
 			(at 179.07 69.85 90)
 			(effects
@@
 			)
 		)
-		(property "LCSC Part #" "C346451"
+		(property "LCSC Part #" "C907989"
 			(at 179.07 69.85 90)
 			(effects
@@
 			)
 		)
-		(property "Max Tolerance" "2%"
+		(property "Max Tolerance" "1%"
 			(at 179.07 69.85 90)
 			(effects

Commit message: optimized clock distribution
Parts:
- removed R125: 0R, Resistor_SMD:R_0603_1608Metric, symbol Device:R
- added C142: 100n, Capacitor_SMD:C_0603_1608Metric, symbol Device:C
Connections:
- net CLK: now also U102.13 (CLK)
- net GNDA: now also C142.2
- net VDDA: now also C142.1
Changed lines of the file:
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@@
 	(title_block
 		(title "MISRC")
-		(date "2025-10-21")
+		(date "2025-10-23")
 		(rev "2.5")
 		(comment 1 "Analog input + ADC")
@@
 	(wire
 		(pts
-			(xy 265.43 105.41) (xy 265.43 127)
+			(xy 265.43 105.41) (xy 265.43 138.43)
 		)
 		(stroke
@@
 	(wire
 		(pts
-			(xy 265.43 134.62) (xy 265.43 138.43)
-		)
-		(stroke
-			(width 0)
-			(type default)
-		)
-	)
-	(wire
-		(pts
 			(xy 220.98 146.05) (xy 220.98 148.59)
 		)
@@
 	)
 	(symbol
-		(lib_id "Device:R")
-		(at 265.43 130.81 0)
-		(unit 1)
-		(exclude_from_sim no)
-		(in_bom yes)
-		(on_board yes)
-		(dnp no)
-		(property "Reference" "R125"
-			(at 265.43 128.27 90)
-			(effects
-				(font
-					(size 1.27 1.27)
-				)
-				(justify right)
-			)
-		)
-		(property "Value" "0R"
-			(at 267.97 129.54 90)
-			(effects
-				(font
-					(size 1.27 1.27)
-				)
-				(justify right)
-			)
-		)
-		(property "Footprint" "Resistor_SMD:R_0603_1608Metric"
-			(at 263.652 130.81 90)
-			(effects
-				(font
-					(size 1.27 1.27)
-				)
-				(hide yes)
-			)
-		)
-		(property "Datasheet" "~"
-			(at 265.43 130.81 0)
-			(effects
-				(font
-					(size 1.27 1.27)
-				)
-				(hide yes)
-			)
-		)
-		(property "Description" ""
-			(at 265.43 130.81 0)
-			(effects
-				(font
-					(size 1.27 1.27)
-				)
-				(hide yes)
-			)
-		)
-		(property "Manufacturer_Part_Number" "0603WAF0000T5E"
-			(at 265.43 130.81 0)
-			(effects
-				(font
-					(size 1.27 1.27)
-				)
-				(hide yes)
-			)
-		)
-		(property "LCSC Part #" "C21189"
-			(at 265.43 130.81 90)
-			(effects
-				(font
-					(size 1.27 1.27)
-				)
-				(hide yes)
-			)
-		)
-		(property "FT Rotation Offset" ""
-			(at 265.43 130.81 90)
-			(effects
-				(font
-					(size 1.27 1.27)
-				)
-				(hide yes)
-			)
-		)
-		(property "Max Tolerance" ""
-			(at 265.43 130.81 90)
-			(effects
-				(font
-					(size 1.27 1.27)
-				)
-				(hide yes)
-			)
-		)
-		(property "Part Selection Note" ""
-			(at 265.43 130.81 90)
-			(effects
-				(font
-					(size 1.27 1.27)
-				)
-				(hide yes)
-			)
-		)
-		(property "Capacitor Ceramic" ""
-			(at 265.43 130.81 90)
-			(effects
-				(font
-					(size 1.27 1.27)
-				)
-				(hide yes)
-			)
-		)
-		(property "Alternative Part" ""
-			(at 265.43 130.81 90)
-			(effects
-				(font
-					(size 1.27 1.27)
-				)
-				(hide yes)
-			)
-		)
-		(pin "1"
-		)
-		(pin "2"
-		)
-		(instances
-			(project "MISRC_v3.0"
-				(path "/bc796fa4-76ff-4554-a44c-2597c6c5788e/f3827713-3b6b-4193-bf1c-3910c26c6fe9"
-					(reference "R125")
-					(unit 1)
-				)
-			)
-		)
-	)
-	(symbol
 		(lib_id "Device:C")
 		(at 113.03 30.48 90)
@@
 	)
 	(symbol
+		(lib_id "Device:C")
+		(at 278.13 39.37 0)
+		(unit 1)
+		(exclude_from_sim no)
+		(in_bom yes)
+		(on_board yes)
+		(dnp no)
+		(fields_autoplaced yes)
+		(property "Reference" "C142"
+			(at 281.94 38.1 0)
+			(effects
+				(font
+					(size 1.27 1.27)
+				)
+				(justify left)
+			)
+		)
+		(property "Value" "100n"
+			(at 281.94 40.64 0)
+			(effects
+				(font
+					(size 1.27 1.27)
+				)
+				(justify left)
+			)
+		)
+		(property "Footprint" "Capacitor_SMD:C_0603_1608Metric"
+			(at 279.0952 43.18 0)
+			(effects
+				(font
+					(size 1.27 1.27)
+				)
+				(hide yes)
+			)
+		)
+		(property "Datasheet" "~"
+			(at 278.13 39.37 0)
+			(effects
+				(font
+					(size 1.27 1.27)
+				)
+				(hide yes)
+			)
+		)
+		(property "Description" ""
+			(at 278.13 39.37 0)
+			(effects
+				(font
+					(size 1.27 1.27)
+				)
+				(hide yes)
+			)
+		)
+		(property "Manufacturer_Part_Number" "CC0603KRX7R9BB104"
+			(at 278.13 39.37 0)
+			(effects
+				(font
+					(size 1.27 1.27)
+				)
+				(hide yes)
+			)
+		)
+		(property "LCSC Part #" "C14663"
+			(at 278.13 39.37 0)
+			(effects
+				(font
+					(size 1.27 1.27)
+				)
+				(hide yes)
+			)
+		)
+		(property "FT Rotation Offset" ""
+			(at 278.13 39.37 0)
+			(effects
+				(font
+					(size 1.27 1.27)
+				)
+				(hide yes)
+			)
+		)
+		(property "Max Tolerance" "10%"
+			(at 278.13 39.37 0)
+			(effects
+				(font
+					(size 1.27 1.27)
+				)
+				(hide yes)
+			)
+		)
+		(property "Part Selection Note" ""
+			(at 278.13 39.37 0)
+			(effects
+				(font
+					(size 1.27 1.27)
+				)
+				(hide yes)
+			)
+		)
+		(property "Capacitor Ceramic" "X7R"
+			(at 278.13 39.37 0)
+			(effects
+				(font
+					(size 1.27 1.27)
+				)
+				(hide yes)
+			)
+		)
+		(property "Alternative Part" ""
+			(at 278.13 39.37 0)
+			(effects
+				(font
+					(size 1.27 1.27)
+				)
+				(hide yes)
+			)
+		)
+		(pin "1"
+		)
+		(pin "2"
+		)
+		(instances
+			(project "misrc_v2.5"
+				(path "/bc796fa4-76ff-4554-a44c-2597c6c5788e/f3827713-3b6b-4193-bf1c-3910c26c6fe9"
+					(reference "C142")
+					(unit 1)
+				)
+			)
+		)
+	)
+	(symbol
 		(lib_id "Device:R")
 		(at 105.41 85.09 90)
@@
 	(symbol
 		(lib_id "power:GNDA")
+		(at 278.13 43.18 0)
+		(unit 1)
+		(exclude_from_sim no)
+		(in_bom yes)
+		(on_board yes)
+		(dnp no)
+		(fields_autoplaced yes)
+		(property "Reference" "#PWR075"
+			(at 278.13 49.53 0)
+			(effects
+				(font
+					(size 1.27 1.27)
+				)
+				(hide yes)
+			)
+		)
+		(property "Value" "GNDA"
+			(at 278.13 48.26 0)
+			(effects
+				(font
+					(size 1.27 1.27)
+				)
+			)
+		)
+		(property "Footprint" ""
+			(at 278.13 43.18 0)
+			(effects
+				(font
+					(size 1.27 1.27)
+				)
+				(hide yes)
+			)
+		)
+		(property "Datasheet" ""
+			(at 278.13 43.18 0)
+			(effects
+				(font
+					(size 1.27 1.27)
+				)
+				(hide yes)
+			)
+		)
+		(property "Description" ""
+			(at 278.13 43.18 0)
+			(effects
+				(font
+					(size 1.27 1.27)
+				)
+				(hide yes)
+			)
+		)
+		(pin "1"
+		)
+		(instances
+			(project "misrc_v2.5"
+				(path "/bc796fa4-76ff-4554-a44c-2597c6c5788e/f3827713-3b6b-4193-bf1c-3910c26c6fe9"
+					(reference "#PWR075")
+					(unit 1)
+				)
+			)
+		)
+	)
+	(symbol
+		(lib_id "power:GNDA")
 		(at 78.74 82.55 0)
 		(mirror x)
@@
 					(unit 1)
 				)
+			)
+		)
+	)
+	(symbol
+		(lib_id "power:VDDA")
+		(at 278.13 35.56 0)
+		(unit 1)
+		(exclude_from_sim no)
+		(in_bom yes)
+		(on_board yes)
+		(dnp no)
+		(fields_autoplaced yes)
+		(property "Reference" "#PWR074"
+			(at 278.13 39.37 0)
+			(effects
+				(font
+					(size 1.27 1.27)
+				)
+				(hide yes)
+			)
+		)
+		(property "Value" "VDDA"
+			(at 278.13 30.48 0)
+			(effects
+				(font
+					(size 1.27 1.27)
+				)
+			)
+		)
+		(property "Footprint" ""
+			(at 278.13 35.56 0)
+			(effects
+				(font
+					(size 1.27 1.27)
+				)
+				(hide yes)
+			)
+		)
+		(property "Datasheet" ""
+			(at 278.13 35.56 0)
+			(effects
+				(font
+					(size 1.27 1.27)
+				)
+				(hide yes)
+			)
+		)
+		(property "Description" ""
+			(at 278.13 35.56 0)
+			(effects
+				(font
+					(size 1.27 1.27)
+				)
+				(hide yes)
+			)
+		)
+		(pin "1"
+		)
+		(instances
+			(project "misrc_v2.5"
+				(path "/bc796fa4-76ff-4554-a44c-2597c6c5788e/f3827713-3b6b-4193-bf1c-3910c26c6fe9"
+					(reference "#PWR074")
+					(unit 1)
+				)

Commit message: fixed zero adjust, more ferrit beads, silkscreen fixes
Parts:
- added C143: 100µ, Capacitor_SMD:C_1210_3225Metric, symbol Device:C
- added C144: 1n/1, Capacitor_SMD:C_0603_1608Metric, symbol Device:C
- added C145, C31: 1µ, Capacitor_SMD:C_0603_1608Metric, symbol Device:C
- added C146, C147: 100n, Capacitor_SMD:C_0603_1608Metric, symbol Device:C
- added FB101: 1k@100MHz,280@10MHz, Inductor_SMD:L_0603_1608Metric, symbol Device:FerriteBead
- added U204: ADA4004-1, Package_TO_SOT_SMD:SOT-23-5, symbol Amplifier_Operational:MCP6001-OT
- R127: value 1kB -> 10; LCSC Part # C110776 -> C22859; Manufacturer_Part_Number RT0603BRD071KL -> 0603WAF100JT5E; Max Tolerance 0.1% -> 1%
Connections:
- net +5VA: now also C147.1, U204.5 (V+)
- net -5VA: now also C146.2, U204.2 (V-)
- net GND: now also C31.2
- net GNDA: now also C143.1, C144.2, C145.2, C146.1, C147.2
- net VDD: now also FB101.1; no longer C126.1, U102.24 (DRVDD)
- net at C127.1, C128.1, R108.2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: now also C143.2
- net at R127.2: now also U204.1, U204.4 (-); no longer RV101.2
- new net: C126.1, C31.1, FB101.2, U102.24 (DRVDD)
- new net: C144.1, C145.1, RV101.2, U204.3 (+)
Other:
- moved on the sheet: C126, C127, C128, R127, RV101
