File: hardware/kicad/dev/input_adc_CH1.kicad_sch (KiCad schematic)
At the start: 91 parts, among them J201 BNC_Rosenberger, J201/2 Conn_01x01_Shielded, J201/3 Conn_Coaxial, SW201 SW_DIP_x04, SW202 SW_DIP_x03, SW203 SW_DIP_x04, SW204 SW_DIP_x03, U201 AD8138ARZ, U202 AD9235

Commit message: changed pot direction
Connections:
- net +5VA: now also RV201.3; no longer RV201.1
- net -5VA: now also RV201.1; no longer RV201.3
Changed lines of the file:
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@@
 	(title_block
 		(title "MISRC")
-		(date "2025-10-10")
+		(date "2025-10-12")
 		(rev "2.5")
 		(comment 1 "Analog input + ADC")
@@
 		(lib_id "Device:R_Potentiometer")
 		(at 48.26 105.41 0)
-		(mirror x)
 		(unit 1)
 		(exclude_from_sim no)
@@
 		)
 		(property "Value" "10k"
-			(at 50.8 107.95 90)
+			(at 50.8 108.204 90)
 			(effects
 				(font
@@
 		)
 		(instances
-			(project "MISRC_v3.0"
+			(project "misrc_v2.5"
 				(path "/bc796fa4-76ff-4554-a44c-2597c6c5788e/56b32eea-16d3-46c8-8e85-f12b91596617"
 					(reference "RV201")

Commit message: updated bom
Parts:
- C201: Manufacturer_Part_Number EMK325ABJ107MM-P -> EMK325ABJ107MM-P
- C218, C219: LCSC Part # C519563 -> C1864402; Manufacturer_Part_Number CC0603FRNPO9BN391 -> GCM1885C2A391FA16D
- C232, C233: LCSC Part # C3895655 -> C3859396; Manufacturer_Name (none) -> Murata; Manufacturer_Part_Number 0603N361F500CT -> GCM1885C2A361FA16D; Mouser Part Number (none) -> 81-GCM1885C2A361FA6D
- C241: Mouser Part Number (none) -> 80-C1812C944J5JLCLTU
- L201, L202: LCSC Part # C346452 -> C2042960; Manufacturer_Part_Number FEC1008CP-R62G-LRH -> LQW2UASR62F00L; Max Tolerance 2% -> 1%
- L203, L204, L205, L206: LCSC Part # C346451 -> C907989; Manufacturer_Part_Number FEC1008CP-R56G-LRH -> LQW2UASR56F00L; Max Tolerance 2% -> 1%
- R207: LCSC Part # C705726 -> C425408; Manufacturer_Part_Number RT0603BRD07150RL -> TC0325B1500T5F
- R219, R220, R221, R222: LCSC Part # C326724 -> C2989449; Manufacturer_Part_Number RT0603BRD0747RL -> TC0325B470JT5F
- SW201, SW203: Mouser Part Number (none) -> 611-SDA04H1SBDR
Changed lines of the file:
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@@
 			)
 		)
-		(property "Manufacturer_Part_Number" "0603N361F500CT"
+		(property "Manufacturer_Part_Number" "GCM1885C2A361FA16D"
 			(at 173.99 55.88 0)
 			(effects
@@
 			)
 		)
-		(property "LCSC Part #" "C3895655"
+		(property "LCSC Part #" "C3859396"
 			(at 173.99 55.88 0)
 			(effects
@@
 			)
 		)
+		(property "Manufacturer_Name" "Murata"
+			(at 173.99 55.88 0)
+			(effects
+				(font
+					(size 1.27 1.27)
+				)
+				(hide yes)
+			)
+		)
+		(property "Mouser Part Number" "81-GCM1885C2A361FA6D"
+			(at 173.99 55.88 0)
+			(effects
+				(font
+					(size 1.27 1.27)
+				)
+				(hide yes)
+			)
+		)
 		(pin "1"
 		)
@@
 			)
 		)
+		(property "Mouser Part Number" "80-C1812C944J5JLCLTU"
+			(at 63.5 73.66 90)
+			(effects
+				(font
+					(size 1.27 1.27)
+				)
+				(hide yes)
+			)
+		)
 		(pin "1"
 		)
@@
 			)
 		)
-		(property "Manufacturer_Part_Number" "0603N361F500CT"
+		(property "Manufacturer_Part_Number" "GCM1885C2A361FA16D"
 			(at 173.99 78.74 0)
 			(effects
@@
 			)
 		)
-		(property "LCSC Part #" "C3895655"
+		(property "LCSC Part #" "C3859396"
 			(at 173.99 78.74 0)
 			(effects
@@
 			)
 		)
+		(property "Manufacturer_Name" "Murata"
+			(at 173.99 78.74 0)
+			(effects
+				(font
+					(size 1.27 1.27)
+				)
+				(hide yes)
+			)
+		)
+		(property "Mouser Part Number" "81-GCM1885C2A361FA6D"
+			(at 173.99 78.74 0)
+			(effects
+				(font
+					(size 1.27 1.27)
+				)
+				(hide yes)
+			)
+		)
 		(pin "1"
 		)
@@
 			)
 		)
-		(property "Manufacturer_Part_Number" "RT0603BRD0747RL"
+		(property "Manufacturer_Part_Number" "TC0325B470JT5F"
 			(at 193.04 64.77 0)
 			(effects
@@
 			)
 		)
-		(property "LCSC Part #" "C326724"
+		(property "LCSC Part #" "C2989449"
 			(at 193.04 64.77 90)
 			(effects
@@
 			)
 		)
-		(property "Manufacturer_Part_Number" "CC0603FRNPO9BN391"
+		(property "Manufacturer_Part_Number" "GCM1885C2A391FA16D"
 			(at 154.94 55.88 0)
 			(effects
@@
 			)
 		)
-		(property "LCSC Part #" "C519563"
+		(property "LCSC Part #" "C1864402"
 			(at 154.94 55.88 0)
 			(effects
@@
 			)
 		)
-		(property "Manufacturer_Part_Number" "RT0603BRD0747RL"
+		(property "Manufacturer_Part_Number" "TC0325B470JT5F"
 			(at 132.08 64.77 0)
 			(effects
@@
 			)
 		)
-		(property "LCSC Part #" "C326724"
+		(property "LCSC Part #" "C2989449"
 			(at 132.08 64.77 90)
 			(effects
@@
 			)
 		)
-		(property "Manufacturer_Part_Number" "FEC1008CP-R56G-LRH"
+		(property "Manufacturer_Part_Number" "LQW2UASR56F00L"
 			(at 180.34 69.85 90)
 			(effects
@@
 			)
 		)
-		(property "LCSC Part #" "C346451"
+		(property "LCSC Part #" "C907989"
 			(at 180.34 69.85 90)
 			(effects
@@
 			)
 		)
-		(property "Max Tolerance" "2%"
+		(property "Max Tolerance" "1%"
 			(at 180.34 69.85 90)
 			(effects
@@
 			)
 		)
-		(property "Manufacturer_Part_Number" "FEC1008CP-R62G-LRH"
+		(property "Manufacturer_Part_Number" "LQW2UASR62F00L"
 			(at 143.51 64.77 90)
 			(effects
@@
 			)
 		)
-		(property "LCSC Part #" "C346452"
+		(property "LCSC Part #" "C2042960"
 			(at 143.51 64.77 90)
 			(effects
@@
 			)
 		)
-		(property "Max Tolerance" "2%"
+		(property "Max Tolerance" "1%"
 			(at 143.51 64.77 90)
 			(effects
@@
 			)
 		)
+		(property "Mouser Part Number" "611-SDA04H1SBDR"
+			(at 55.88 44.45 90)
+			(effects
+				(font
+					(size 1.27 1.27)
+				)
+				(hide yes)
+			)
+		)
 		(pin "1"
 		)
@@
 			)
 		)
-		(property "Manufacturer_Part_Number" "CC0603FRNPO9BN391"
+		(property "Manufacturer_Part_Number" "GCM1885C2A391FA16D"
 			(at 154.94 78.74 0)
 			(effects
@@
 			)
 		)
-		(property "LCSC Part #" "C519563"
+		(property "LCSC Part #" "C1864402"
 			(at 154.94 78.74 0)
 			(effects
@@
 			)
 		)
-		(property "Manufacturer_Part_Number" "FEC1008CP-R56G-LRH"
+		(property "Manufacturer_Part_Number" "LQW2UASR56F00L"
 			(at 167.64 64.77 90)
 			(effects
@@
 			)
 		)
-		(property "LCSC Part #" "C346451"
+		(property "LCSC Part #" "C907989"
 			(at 167.64 64.77 90)
 			(effects
@@
 			)
 		)
-		(property "Max Tolerance" "2%"
+		(property "Max Tolerance" "1%"
 			(at 167.64 64.77 90)
 			(effects
@@
 			)
 		)
-		(property "Manufacturer_Part_Number" "FEC1008CP-R56G-LRH"
+		(property "Manufacturer_Part_Number" "LQW2UASR56F00L"
 			(at 167.64 69.85 90)
 			(effects
@@
 			)
 		)
-		(property "LCSC Part #" "C346451"
+		(property "LCSC Part #" "C907989"
 			(at 167.64 69.85 90)
 			(effects
@@
 			)
 		)
-		(property "Max Tolerance" "2%"
+		(property "Max Tolerance" "1%"
 			(at 167.64 69.85 90)
 			(effects
@@
 			)
 		)
-		(property "Manufacturer_Part_Number" "RT0603BRD07150RL"
+		(property "Manufacturer_Part_Number" "TC0325B1500T5F"
 			(at 85.09 78.74 0)
 			(effects
@@
 			)
 		)
-		(property "LCSC Part #" "C705726"
+		(property "LCSC Part #" "C425408"
 			(at 85.09 78.74 90)
 			(effects
@@
 			)
 		)
-		(property "Manufacturer_Part_Number" "FEC1008CP-R62G-LRH"
+		(property "Manufacturer_Part_Number" "LQW2UASR62F00L"
 			(at 143.51 69.85 90)
 			(effects
@@
 			)
 		)
-		(property "LCSC Part #" "C346452"
+		(property "LCSC Part #" "C2042960"
 			(at 143.51 69.85 90)
 			(effects
@@
 			)
 		)
-		(property "Max Tolerance" "2%"
+		(property "Max Tolerance" "1%"
 			(at 143.51 69.85 90)
 			(effects
@@
 			)
 		)
+		(property "Mouser Part Number" "611-SDA04H1SBDR"
+			(at 119.38 45.72 90)
+			(effects
+				(font
+					(size 1.27 1.27)
+				)
+				(hide yes)
+			)
+		)
 		(pin "1"
 		)
@@
 			)
 		)
-		(property "Manufacturer_Part_Number" "RT0603BRD0747RL"
+		(property "Manufacturer_Part_Number" "TC0325B470JT5F"
 			(at 132.08 69.85 0)
 			(effects
@@
 			)
 		)
-		(property "LCSC Part #" "C326724"
+		(property "LCSC Part #" "C2989449"
 			(at 132.08 69.85 90)
 			(effects
@@
 			)
 		)
-		(property "Manufacturer_Part_Number" "FEC1008CP-R56G-LRH"
+		(property "Manufacturer_Part_Number" "LQW2UASR56F00L"
 			(at 180.34 64.77 90)
 			(effects
@@
 			)
 		)
-		(property "LCSC Part #" "C346451"
+		(property "LCSC Part #" "C907989"
 			(at 180.34 64.77 90)
 			(effects
@@
 			)
 		)
-		(property "Max Tolerance" "2%"
+		(property "Max Tolerance" "1%"
 			(at 180.34 64.77 90)
 			(effects
@@
 			)
 		)
-		(property "Manufacturer_Part_Number" " EMK325ABJ107MM-P"
+		(property "Manufacturer_Part_Number" "EMK325ABJ107MM-P"
 			(at 41.91 63.5 0)
 			(effects
@@
 			)
 		)
-		(property "Manufacturer_Part_Number" "RT0603BRD0747RL"
+		(property "Manufacturer_Part_Number" "TC0325B470JT5F"
 			(at 193.04 69.85 0)
 			(effects
@@
 			)
 		)
-		(property "LCSC Part #" "C326724"
+		(property "LCSC Part #" "C2989449"
 			(at 193.04 69.85 90)
 			(effects

Commit message: optimized clock distribution
Parts:
- removed R225: 0R, Resistor_SMD:R_0603_1608Metric, symbol Device:R
- added C242: 100n, Capacitor_SMD:C_0603_1608Metric, symbol Device:C
Connections:
- net CLK: now also U202.13 (CLK)
- net GNDA: now also C242.2
- net VDDA: now also C242.1
Changed lines of the file:
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@@
 	(title_block
 		(title "MISRC")
-		(date "2025-10-21")
+		(date "2025-10-23")
 		(rev "2.5")
 		(comment 1 "Analog input + ADC")
@@
 	(wire
 		(pts
-			(xy 266.7 107.95) (xy 266.7 129.54)
+			(xy 266.7 107.95) (xy 266.7 140.97)
 		)
 		(stroke
@@
 	(wire
 		(pts
-			(xy 266.7 137.16) (xy 266.7 140.97)
-		)
-		(stroke
-			(width 0)
-			(type default)
-		)
-	)
-	(wire
-		(pts
 			(xy 222.25 148.59) (xy 222.25 151.13)
 		)
@@
 	)
 	(symbol
+		(lib_id "Device:C")
+		(at 275.59 39.37 0)
+		(unit 1)
+		(exclude_from_sim no)
+		(in_bom yes)
+		(on_board yes)
+		(dnp no)
+		(fields_autoplaced yes)
+		(property "Reference" "C242"
+			(at 279.4 38.1 0)
+			(effects
+				(font
+					(size 1.27 1.27)
+				)
+				(justify left)
+			)
+		)
+		(property "Value" "100n"
+			(at 279.4 40.64 0)
+			(effects
+				(font
+					(size 1.27 1.27)
+				)
+				(justify left)
+			)
+		)
+		(property "Footprint" "Capacitor_SMD:C_0603_1608Metric"
+			(at 276.5552 43.18 0)
+			(effects
+				(font
+					(size 1.27 1.27)
+				)
+				(hide yes)
+			)
+		)
+		(property "Datasheet" "~"
+			(at 275.59 39.37 0)
+			(effects
+				(font
+					(size 1.27 1.27)
+				)
+				(hide yes)
+			)
+		)
+		(property "Description" ""
+			(at 275.59 39.37 0)
+			(effects
+				(font
+					(size 1.27 1.27)
+				)
+				(hide yes)
+			)
+		)
+		(property "Manufacturer_Part_Number" "CC0603KRX7R9BB104"
+			(at 275.59 39.37 0)
+			(effects
+				(font
+					(size 1.27 1.27)
+				)
+				(hide yes)
+			)
+		)
+		(property "LCSC Part #" "C14663"
+			(at 275.59 39.37 0)
+			(effects
+				(font
+					(size 1.27 1.27)
+				)
+				(hide yes)
+			)
+		)
+		(property "FT Rotation Offset" ""
+			(at 275.59 39.37 0)
+			(effects
+				(font
+					(size 1.27 1.27)
+				)
+				(hide yes)
+			)
+		)
+		(property "Max Tolerance" "10%"
+			(at 275.59 39.37 0)
+			(effects
+				(font
+					(size 1.27 1.27)
+				)
+				(hide yes)
+			)
+		)
+		(property "Part Selection Note" ""
+			(at 275.59 39.37 0)
+			(effects
+				(font
+					(size 1.27 1.27)
+				)
+				(hide yes)
+			)
+		)
+		(property "Capacitor Ceramic" "X7R"
+			(at 275.59 39.37 0)
+			(effects
+				(font
+					(size 1.27 1.27)
+				)
+				(hide yes)
+			)
+		)
+		(property "Alternative Part" ""
+			(at 275.59 39.37 0)
+			(effects
+				(font
+					(size 1.27 1.27)
+				)
+				(hide yes)
+			)
+		)
+		(pin "1"
+		)
+		(pin "2"
+		)
+		(instances
+			(project "misrc_v2.5"
+				(path "/bc796fa4-76ff-4554-a44c-2597c6c5788e/56b32eea-16d3-46c8-8e85-f12b91596617"
+					(reference "C242")
+					(unit 1)
+				)
+			)
+		)
+	)
+	(symbol
 		(lib_id "power:+5VA")
 		(at 226.06 35.56 0)
@@
 	)
 	(symbol
+		(lib_id "power:VDDA")
+		(at 275.59 35.56 0)
+		(unit 1)
+		(exclude_from_sim no)
+		(in_bom yes)
+		(on_board yes)
+		(dnp no)
+		(fields_autoplaced yes)
+		(property "Reference" "#PWR072"
+			(at 275.59 39.37 0)
+			(effects
+				(font
+					(size 1.27 1.27)
+				)
+				(hide yes)
+			)
+		)
+		(property "Value" "VDDA"
+			(at 275.59 30.48 0)
+			(effects
+				(font
+					(size 1.27 1.27)
+				)
+			)
+		)
+		(property "Footprint" ""
+			(at 275.59 35.56 0)
+			(effects
+				(font
+					(size 1.27 1.27)
+				)
+				(hide yes)
+			)
+		)
+		(property "Datasheet" ""
+			(at 275.59 35.56 0)
+			(effects
+				(font
+					(size 1.27 1.27)
+				)
+				(hide yes)
+			)
+		)
+		(property "Description" ""
+			(at 275.59 35.56 0)
+			(effects
+				(font
+					(size 1.27 1.27)
+				)
+				(hide yes)
+			)
+		)
+		(pin "1"
+		)
+		(instances
+			(project "misrc_v2.5"
+				(path "/bc796fa4-76ff-4554-a44c-2597c6c5788e/56b32eea-16d3-46c8-8e85-f12b91596617"
+					(reference "#PWR072")
+					(unit 1)
+				)
+			)
+		)
+	)
+	(symbol
 		(lib_id "Device:R")
 		(at 193.04 64.77 90)
@@
 	)
 	(symbol
+		(lib_id "power:GNDA")
+		(at 275.59 43.18 0)
+		(unit 1)
+		(exclude_from_sim no)
+		(in_bom yes)
+		(on_board yes)
+		(dnp no)
+		(fields_autoplaced yes)
+		(property "Reference" "#PWR073"
+			(at 275.59 49.53 0)
+			(effects
+				(font
+					(size 1.27 1.27)
+				)
+				(hide yes)
+			)
+		)
+		(property "Value" "GNDA"
+			(at 275.59 48.26 0)
+			(effects
+				(font
+					(size 1.27 1.27)
+				)
+			)
+		)
+		(property "Footprint" ""
+			(at 275.59 43.18 0)
+			(effects
+				(font
+					(size 1.27 1.27)
+				)
+				(hide yes)
+			)
+		)
+		(property "Datasheet" ""
+			(at 275.59 43.18 0)
+			(effects
+				(font
+					(size 1.27 1.27)
+				)
+				(hide yes)
+			)
+		)
+		(property "Description" ""
+			(at 275.59 43.18 0)
+			(effects
+				(font
+					(size 1.27 1.27)
+				)
+				(hide yes)
+			)
+		)
+		(pin "1"
+		)
+		(instances
+			(project "misrc_v2.5"
+				(path "/bc796fa4-76ff-4554-a44c-2597c6c5788e/56b32eea-16d3-46c8-8e85-f12b91596617"
+					(reference "#PWR073")
+					(unit 1)
+				)
+			)
+		)
+	)
+	(symbol
 		(lib_id "Device:C")
 		(at 39.37 87.63 0)
@@
 					(unit 1)
 				)
-			)
-		)
-	)
-	(symbol
-		(lib_id "Device:R")
-		(at 266.7 133.35 0)
-		(unit 1)
-		(exclude_from_sim no)
-		(in_bom yes)
-		(on_board yes)
-		(dnp no)
-		(property "Reference" "R225"
-			(at 266.7 130.81 90)
-			(effects
-				(font
-					(size 1.27 1.27)
-				)
-				(justify right)
-			)
-		)
-		(property "Value" "0R"
-			(at 269.24 132.08 90)
-			(effects
-				(font
-					(size 1.27 1.27)
-				)
-				(justify right)
-			)
-		)
-		(property "Footprint" "Resistor_SMD:R_0603_1608Metric"
-			(at 264.922 133.35 90)
-			(effects
-				(font
-					(size 1.27 1.27)
-				)
-				(hide yes)
-			)
-		)
-		(property "Datasheet" "~"
-			(at 266.7 133.35 0)
-			(effects
-				(font
-					(size 1.27 1.27)
-				)
-				(hide yes)
-			)
-		)
-		(property "Description" ""
-			(at 266.7 133.35 0)
-			(effects
-				(font
-					(size 1.27 1.27)
-				)
-				(hide yes)
-			)
-		)
-		(property "Manufacturer_Part_Number" "0603WAF0000T5E"
-			(at 266.7 133.35 0)
-			(effects
-				(font
-					(size 1.27 1.27)
-				)
-				(hide yes)
-			)
-		)
-		(property "LCSC Part #" "C21189"
-			(at 266.7 133.35 90)
-			(effects
-				(font
-					(size 1.27 1.27)
-				)
-				(hide yes)
-			)
-		)
-		(property "FT Rotation Offset" ""
-			(at 266.7 133.35 90)
-			(effects
-				(font
-					(size 1.27 1.27)
-				)
-				(hide yes)
-			)
-		)
-		(property "Max Tolerance" ""
-			(at 266.7 133.35 90)
-			(effects
-				(font
-					(size 1.27 1.27)
-				)
-				(hide yes)
-			)
-		)
-		(property "Part Selection Note" ""
-			(at 266.7 133.35 90)
-			(effects
-				(font
-					(size 1.27 1.27)
-				)
-				(hide yes)
-			)
-		)
-		(property "Capacitor Ceramic" ""
-			(at 266.7 133.35 90)
-			(effects
-				(font
-					(size 1.27 1.27)
-				)
-				(hide yes)
-			)
-		)
-		(property "Alternative Part" ""
-			(at 266.7 133.35 90)
-			(effects
-				(font
-					(size 1.27 1.27)
-				)
-				(hide yes)
-			)
-		)
-		(pin "1"
-		)
-		(pin "2"
-		)
-		(instances
-			(project "MISRC_v3.0"
-				(path "/bc796fa4-76ff-4554-a44c-2597c6c5788e/56b32eea-16d3-46c8-8e85-f12b91596617"
-					(reference "R225")
-					(unit 1)
-				)

Commit message: fixed zero adjust, more ferrit beads, silkscreen fixes
Parts:
- added C2, C245: 1µ, Capacitor_SMD:C_0603_1608Metric, symbol Device:C
- added C243: 100µ, Capacitor_SMD:C_1210_3225Metric, symbol Device:C
- added C244: 1n/1, Capacitor_SMD:C_0603_1608Metric, symbol Device:C
- added C246, C247: 100n, Capacitor_SMD:C_0603_1608Metric, symbol Device:C
- added FB201: 1k@100MHz,280@10MHz, Inductor_SMD:L_0603_1608Metric, symbol Device:FerriteBead
- added U203: ADA4004-1, Package_TO_SOT_SMD:SOT-23-5, symbol Amplifier_Operational:MCP6001-OT
- R227: value 1kB -> 10; LCSC Part # C110776 -> C22859; Manufacturer_Part_Number RT0603BRD071KL -> 0603WAF100JT5E; Max Tolerance 0.1% -> 1%
Connections:
- net +5VA: now also C247.1, U203.5 (V+)
- net -5VA: now also C246.2, U203.2 (V-)
- net GND: now also C2.2
- net GNDA: now also C243.1, C244.2, C245.2, C246.1, C247.2
- net VDD: now also FB201.1; no longer C226.1, U202.24 (DRVDD)
- net at C227.1, C228.1, R208.2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: now also C243.2
- net at R227.2: now also U203.1, U203.4 (-); no longer RV201.2
- new net: C2.1, C226.1, FB201.2, U202.24 (DRVDD)
- new net: C244.1, C245.1, RV201.2, U203.3 (+)
Other:
- moved on the sheet: C226, C227, C228, R227, RV201
