File: hardware/kicad/dev/power_supply.kicad_sch (KiCad schematic)
At the start: 35 parts, among them Q1 FZT690B, Q2 FZT790A, U6 LM2662, U7 LT3042xMSE

Commit message: updated bom
Parts:
- C10, C11, C16, C17, C18, C19, C6: Capacitor Ceramic (none) -> Polymer; Manufacturer_Name (none) -> Panasonic; Mouser Part Number (none) -> 667-16SVPF1000M
- L1, L2: Manufacturer_Name (none) -> Bourns; Mouser Part Number (none) -> 652-SRU8043-101Y
Changed lines of the file:
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@@
 			)
 		)
-		(property "Capacitor Ceramic" ""
+		(property "Capacitor Ceramic" "Polymer"
 			(at 111.76 74.93 0)
 			(effects
@@
 			)
 		)
+		(property "Manufacturer_Name" "Panasonic"
+			(at 111.76 74.93 0)
+			(effects
+				(font
+					(size 1.27 1.27)
+				)
+				(hide yes)
+			)
+		)
+		(property "Mouser Part Number" "667-16SVPF1000M"
+			(at 111.76 74.93 0)
+			(effects
+				(font
+					(size 1.27 1.27)
+				)
+				(hide yes)
+			)
+		)
 		(pin "1"
 		)
@@
 			)
 		)
+		(property "Manufacturer_Name" "Bourns"
+			(at 74.93 63.5 90)
+			(effects
+				(font
+					(size 1.27 1.27)
+				)
+				(hide yes)
+			)
+		)
+		(property "Mouser Part Number" "652-SRU8043-101Y"
+			(at 74.93 63.5 90)
+			(effects
+				(font
+					(size 1.27 1.27)
+				)
+				(hide yes)
+			)
+		)
 		(pin "1"
 		)
@@
 			)
 		)
-		(property "Capacitor Ceramic" ""
+		(property "Capacitor Ceramic" "Polymer"
 			(at 83.82 72.39 0)
 			(effects
@@
 			)
 		)
+		(property "Manufacturer_Name" "Panasonic"
+			(at 83.82 72.39 0)
+			(effects
+				(font
+					(size 1.27 1.27)
+				)
+				(hide yes)
+			)
+		)
+		(property "Mouser Part Number" "667-16SVPF1000M"
+			(at 83.82 72.39 0)
+			(effects
+				(font
+					(size 1.27 1.27)
+				)
+				(hide yes)
+			)
+		)
 		(pin "1"
 		)
@@
 			)
 		)
+		(property "Manufacturer_Name" "Bourns"
+			(at 63.5 36.83 90)
+			(effects
+				(font
+					(size 1.27 1.27)
+				)
+				(hide yes)
+			)
+		)
+		(property "Mouser Part Number" "652-SRU8043-101Y"
+			(at 63.5 36.83 90)
+			(effects
+				(font
+					(size 1.27 1.27)
+				)
+				(hide yes)
+			)
+		)
 		(pin "1"
 		)
@@
 			)
 		)
-		(property "Capacitor Ceramic" ""
+		(property "Capacitor Ceramic" "Polymer"
 			(at 119.38 72.39 0)
 			(effects
@@
 			)
 		)
+		(property "Manufacturer_Name" "Panasonic"
+			(at 119.38 72.39 0)
+			(effects
+				(font
+					(size 1.27 1.27)
+				)
+				(hide yes)
+			)
+		)
+		(property "Mouser Part Number" "667-16SVPF1000M"
+			(at 119.38 72.39 0)
+			(effects
+				(font
+					(size 1.27 1.27)
+				)
+				(hide yes)
+			)
+		)
 		(pin "1"
 		)
@@
 			)
 		)
-		(property "Capacitor Ceramic" ""
+		(property "Capacitor Ceramic" "Polymer"
 			(at 107.95 45.72 0)
 			(effects
@@
 			)
 		)
+		(property "Manufacturer_Name" "Panasonic"
+			(at 107.95 45.72 0)
+			(effects
+				(font
+					(size 1.27 1.27)
+				)
+				(hide yes)
+			)
+		)
+		(property "Mouser Part Number" "667-16SVPF1000M"
+			(at 107.95 45.72 0)
+			(effects
+				(font
+					(size 1.27 1.27)
+				)
+				(hide yes)
+			)
+		)
 		(pin "1"
 		)
@@
 			)
 		)
-		(property "Capacitor Ceramic" ""
+		(property "Capacitor Ceramic" "Polymer"
 			(at 72.39 45.72 0)
 			(effects
@@
 			)
 		)
+		(property "Manufacturer_Name" "Panasonic"
+			(at 72.39 45.72 0)
+			(effects
+				(font
+					(size 1.27 1.27)
+				)
+				(hide yes)
+			)
+		)
+		(property "Mouser Part Number" "667-16SVPF1000M"
+			(at 72.39 45.72 0)
+			(effects
+				(font
+					(size 1.27 1.27)
+				)
+				(hide yes)
+			)
+		)
 		(pin "1"
 		)
@@
 			)
 		)
-		(property "Capacitor Ceramic" ""
+		(property "Capacitor Ceramic" "Polymer"
 			(at 100.33 48.26 0)
 			(effects
@@
 			)
 		)
+		(property "Manufacturer_Name" "Panasonic"
+			(at 100.33 48.26 0)
+			(effects
+				(font
+					(size 1.27 1.27)
+				)
+				(hide yes)
+			)
+		)
+		(property "Mouser Part Number" "667-16SVPF1000M"
+			(at 100.33 48.26 0)
+			(effects
+				(font
+					(size 1.27 1.27)
+				)
+				(hide yes)
+			)
+		)
 		(pin "1"
 		)
@@
 			)
 		)
-		(property "Capacitor Ceramic" ""
+		(property "Capacitor Ceramic" "Polymer"
 			(at 48.26 45.72 0)
 			(effects
@@
 			(at 48.26 45.72 0)
 			(effects
+				(font
+					(size 1.27 1.27)
+				)
+				(hide yes)
+			)
+		)
+		(property "Manufacturer_Name" "Panasonic"
+			(at 48.26 45.72 0)
+			(effects
+				(font
+					(size 1.27 1.27)
+				)
+				(hide yes)
+			)
+		)
+		(property "Mouser Part Number" "667-16SVPF1000M"
+			(at 48.26 45.72 0)
+			(effects
